File: Kicad/servo/servo.kicad_sch (KiCad schematic)
At the start: 12 parts, among them J1 pwm, J2 servo, J3 servo, J4 servo, J5 servo, P1 XT60

Commit message: servo回路作成＆PCB用
Parts:
- added J6: servo5, Connector_PinHeader_2.54mm:PinHeader_1x03_P2.54mm_Vertical, symbol Connector:Conn_01x03_Pin
- added R5: 220Ω, Resistor_THT:R_Axial_DIN0207_L6.3mm_D2.5mm_P7.62mm_Horizontal, symbol Device:R
- J2: value servo -> servo1
- J3: value servo -> servo2
- J4: value servo -> servo3
- J5: value servo -> servo4
- P1: value XT60 -> XT30; footprint Connector_AMASS:AMASS_XT60PW-M_1x02_P7.20mm_Horizontal -> Connector_AMASS:AMASS_XT30PW-M_1x02_P2.50mm_Horizontal
Connections:
- net +5V: now also P1.2 (Pin_2), J6.2 (Pin_2); no longer J1.5 (Pin_5), P1.1 (Pin_1)
- net GND: now also J1.1 (Pin_1), J2.1 (Pin_1), J3.1 (Pin_1), J4.1 (Pin_1), J5.1 (Pin_1), P1.1 (Pin_1), J6.1 (Pin_1); no longer J1.6 (Pin_6), J2.3 (Pin_3), J3.3 (Pin_3), J4.3 (Pin_3), J5.3 (Pin_3), P1.2 (Pin_2)
- net at R4.2: now also J3.3 (Pin_3); no longer J5.1 (Pin_1)
- net at R3.2: now also J4.3 (Pin_3); no longer J4.1 (Pin_1)
- net at R1.1: now also J1.6 (Pin_6); no longer J1.1 (Pin_1)
- net at J1.2 (Pin_2): now also R5.1; no longer R2.1
- net at J1.3 (Pin_3): now also R4.1; no longer R3.1
- net at J1.4 (Pin_4): now also R3.1; no longer R4.1
- net at R2.2: now also J5.3 (Pin_3); no longer J3.1 (Pin_1)
- net at R1.2: now also J6.3 (Pin_3); no longer J2.1 (Pin_1)
- new net: J1.5 (Pin_5), R2.1
- new net: J2.3 (Pin_3), R5.2
Other:
- moved on the sheet: J1, J2, J3, J4, J5, P1

Commit message: 最新回路基盤　動作表示用LEDもつけた
Parts:
- added D1: LED, LED_THT:LED_D3.0mm, symbol Device:LED
- added R6: 1kΩ, Resistor_THT:R_Axial_DIN0207_L6.3mm_D2.5mm_P7.62mm_Horizontal, symbol Device:R
Connections:
- net GND: now also D1.1 (K)
- net +5V renamed V_SERVO
- net V_SERVO: now also R6.1
- new net: D1.2 (A), R6.2
