File: Kicad/ESP/ESP.kicad_sch (KiCad schematic)
At the start: 0 parts

Commit message: 回路完成
Parts:
- added D1: CAN_STATUS_LED_GPIO, LED_THT:LED_D3.0mm, symbol Device:LED
- added D2: LOWER_ARM_STATUS_LED_GPIO, LED_THT:LED_D3.0mm, symbol Device:LED
- added D3: UPPER_ARM_STATUS_LED_GPIO, LED_THT:LED_D3.0mm, symbol Device:LED
- added D4: ROBOMAS_CONTROLLER_STATUS_LED_GPIO, LED_THT:LED_D3.0mm, symbol Device:LED
- added D5: CONTROLLER_1_LED_GPIO, LED_THT:LED_D3.0mm, symbol Device:LED
- added D6: CONTROLLER_2_LED_GPIO, LED_THT:LED_D3.0mm, symbol Device:LED
- added D7: STATUS_LED_GPIO, LED_THT:LED_D3.0mm, symbol Device:LED
- added H1, H2, H3, H4: MountingHole, MountingHole:MountingHole_3.2mm_M3, symbol Mechanical:MountingHole
- added J1: 5V, Connector_PinHeader_2.54mm:PinHeader_1x02_P2.54mm_Vertical, symbol Connector:Conn_01x02_Pin
- added J2: CAN, Connector_PinHeader_2.54mm:PinHeader_1x05_P2.54mm_Vertical, symbol Connector:Conn_01x05_Pin
- added J3: 3V3, Connector_PinHeader_2.54mm:PinHeader_1x02_P2.54mm_Vertical, symbol Connector:Conn_01x02_Pin
- added R1, R2, R3, R4, R5, R6, R7: 300R, Resistor_THT:R_Axial_DIN0207_L6.3mm_D2.5mm_P7.62mm_Horizontal, symbol Device:R
- added U1: ESP32_DevKitC-32E, ESP32_DevKitC_32E:ESP32_DevKitC_32E, symbol ESP32_DevKitC_32E:ESP32_DevKitC_32E
Connections:
- new net: D3.2 (A), R3.2
- new net: D5.2 (A), R5.2
- new net: D6.2 (A), R6.2
- new net: D2.2 (A), R2.2
- new net: D1.2 (A), R1.2
- new net: D4.2 (A), R4.2
- new net: D7.2 (A), R7.2
- new net +3.3V: J2.5 (Pin_5), J3.2 (Pin_2), U1.1 (3V3)
- new net +5V: J1.2 (Pin_2), J2.4 (Pin_4), U1.19 (5V)
- new net CAN_RX: J2.2 (Pin_2), U1.22 (GPIO22)
- new net CAN_STATUS_LED_GPIO: R1.1, U1.9 (GPIO25)
- new net CAN_TX: J2.3 (Pin_3), U1.25 (GPIO21)
- new net CONTROLLER_1_LED_GPIO: R5.1, U1.32 (GPIO4)
- new net CONTROLLER_2_LED_GPIO: R6.1, U1.28 (GPIO18)
- new net GND: D1.1 (K), D2.1 (K), D3.1 (K), D4.1 (K), D5.1 (K), D6.1 (K), D7.1 (K), J1.1 (Pin_1), J2.1 (Pin_1), J3.1 (Pin_1), U1.[14,20,26] (GND)
- new net LOWER_ARM_STATUS_LED_GPIO: R2.1, U1.10 (GPIO26)
- new net ROBOMAS_CONTROLLER_STATUS_LED_GPIO: R4.1, U1.7 (GPIO32)
- new net STATUS_LED_GPIO: R7.1, U1.8 (GPIO33)
- new net UPPER_ARM_STATUS_LED_GPIO: R3.1, U1.11 (GPIO27)
- no-connect marks 0 -> 24
